File: KiCad Files/Controller PCB/Controller_PCB.kicad_pcb (KiCad board)
At the start: 2 copper layers, 69.9 x 59.2 mm, 19 parts, among them J1 0532610271, J2 5037630291, J3 0532610271, J4 5051100592, J5 5051100592, J7 5051101892, U1 GC+2.0

Commit message: Add files via upload
Parts:
- removed the G*** at (170.4, 101.9)
- moved G*** 4.93 mm to (174.0, 100.5)
Other:
- board text added: "REV 2.1 - 27/5/2026"
- board text removed: "REV 2.0 - 15/11/2025"
