File: KiCad Files/Main PCB/Main PCB.kicad_pcb (KiCad board)
At the start: 4 copper layers, 81.5 x 134.5 mm, 38 parts, among them J1 5051104091, J2 5051105091, J21 5037630291, J22 5040500791, J23 5051100892, J25 SJ-3524-SMT, J3 Conn_02x08_Counter_Clockwise, J4 Conn_02x10_Counter_Clockwise, J5 Conn_01x01_Pin, J6 Conn_01x01_Pin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

Commit message: Add files via upload
Parts:
- removed the G*** at (81.0, 38.1)
- moved G*** 6.99 mm to (85.6, 34.7)
Other:
- board text added: "REV 2.1 - 27/5/2026"
- board text removed: "REV 2.0 - 15/11/2025"
