File: KiCad Files/Shielded FFC/Shileded FFC.kicad_pcb (KiCad board)
At the start: 2 copper layers, 20.5 x 35 mm, 5 parts, among them J1 Conn_01x40_Pin, J2 Conn_01x40_Pin

Commit message: Add files via upload
Parts:
- removed the G*** at (155.3, 74.2)
Other:
- board text added: "Xii-Boy Ultra FFC XBU-006 | REV 2.1 | 27/5/2026"
- board text removed: "Xii-Boy Ultra FFC XBU-006 | REV 2.0 | 15/11/2025"
