File: KiCad Files/Trigger PCB/Trigger PCB.kicad_pcb (KiCad board)
At the start: 2 copper layers, 51.6 x 23.1 mm, 8 parts, among them J1 5051100592, J2 5051100892, J3 5051100592

Commit message: Add files via upload
Parts:
- removed the G*** at (145.5, 84.6)
- moved G*** 34.6 mm to (113.4, 68.4)
Other:
- board text added: "REV 2.1 - 27/5/2026"
- board text removed: "REV 2.0 - 15/11/2025"
