File: KiCad Files/Xii-DD/Xii-DD.kicad_pcb (KiCad board)
At the start: 2 copper layers, 82 x 71.6 mm, 6 parts, among them J1 5051104091, J3 5051101892

Commit message: Add files via upload
Parts:
- removed the G*** at (152.3, 111.6)
- moved G*** 4.63 mm to (151.3, 115.7)
Other:
- board text added: "XBU-002 REV 2.1 - 27/5/2026"
- board text removed: "XBU-002 REV 2.0 - 15/11/2025"
