File: KiCad Files/Xii-Flex Ultra/Xii-Flex Ultra.kicad_pcb (KiCad board)
At the start: 2 copper layers, 49.8 x 54.7 mm, 4 parts, among them J1 Conn_01x50_Pin

Commit message: Add files via upload
Parts:
- removed the G*** at (148.1, 116.0)
Other:
- board text added: "REV 2.1 - 27/5/2026"
- board text removed: "REV 2.0 - 15/11/2025"
