File: KiCad Files/Xii-Flex Ultra/Xii-Flex Ultra.kicad_pcb (KiCad board)
At the start: 2 copper layers, 49.8 x 54.7 mm, 3 parts, among them J1 Conn_01x50_Pin

Commit message: Add files via upload
Other:
- board text added: "REV 2.2 - 20/7/2026CH"
- board text removed: "REV 2.1 - 27/5/2026"
Changed lines of the file:
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@@
 		)
 	)
-	(gr_text "REV 2.1 - 27/5/2026"
+	(gr_text "REV 2.2 - 20/7/2026CH"
 		(at 139.98 120.93 0)
 		(layer "F.SilkS")
